Commit message: updated urdf

File: hopper.urdf (robot description, URDF)
Before this commit: robot 2D_Hopper, 4 links, 3 joints
Links:
- added link leg_theta
- added link leg_x
- added link leg_y
Joints:
- removed joint leg
- added joint legtheta: type continuous, parent leg_theta, child leg, axis 0 1 0
- added joint legx: type prismatic, parent ground, child leg_x, axis 1 0 0
- added joint legy: type prismatic, parent leg_x, child leg_y, axis 0 0 1

Commit message: fixed links

File: hopper.urdf (robot description, URDF)
Before this commit: robot 2D_Hopper, 7 links, 5 joints
Links:
- removed link leg_theta
Joints:
- joint legtheta: parent leg_theta -> leg_y

Commit message: added ground to world connection

File: hopper.urdf (robot description, URDF)
Before this commit: robot 2D_Hopper, 6 links, 5 joints
Joints:
- added joint ground_is_world: type fixed, parent , child 

Commit message: link not name. whoops.

File: hopper.urdf (robot description, URDF)
Before this commit: robot 2D_Hopper, 6 links, 6 joints
Joints:
- joint ground_is_world: child  -> ground; parent  -> world

Commit message: made ground bigger

File: hopper.urdf (robot description, URDF)
Before this commit: robot 2D_Hopper, 6 links, 6 joints
Links:
- link ground: geometry collision box size=100 1 2; visual box size=100 1 2

Commit message: changed inertia of leg

File: hopper.urdf (robot description, URDF)
Before this commit: robot 2D_Hopper, 6 links, 6 joints
Links:
- link leg: mass 10 -> 1

Commit message: switched + and - for leg spring, works now?

File: hopper.urdf (robot description, URDF)
Before this commit: robot 2D_Hopper, 6 links, 6 joints
Joints:
- joint z0: axis 0 0 1 -> 0 0 -1

Commit message: fixed auto collision between slide and leg hopefully

File: hopper.urdf (robot description, URDF)
Before this commit: robot 2D_Hopper, 6 links, 6 joints
Links:
- link leg: geometry collision box size=0.05 0.2 0.05; collision box size=0.2 0.2 .1

Commit message: trying stuff

File: hopper.urdf (robot description, URDF)
Before this commit: robot 2D_Hopper, 6 links, 6 joints
Joints:
- joint z0: axis 0 0 -1 -> 0 0 1

Commit message: flipped parent and child in prismatic joint

File: hopper.urdf (robot description, URDF)
Before this commit: robot 2D_Hopper, 6 links, 6 joints
Joints:
- joint z0: child slide -> leg; parent leg -> slide

Commit message: reverted. damn

File: hopper.urdf (robot description, URDF)
Before this commit: robot 2D_Hopper, 6 links, 6 joints
Joints:
- joint z0: child leg -> slide; parent slide -> leg

Commit message: removed all collisions except for ground and toe

File: hopper.urdf (robot description, URDF)
Before this commit: robot 2D_Hopper, 6 links, 6 joints
Links:
- link leg: geometry collision box size=0.05 0.2 0.05; visual box size=0.05 0.2 1.1

Commit message: added y limit in joint. maybe that works better than collision?

File: hopper.urdf (robot description, URDF)
Before this commit: robot 2D_Hopper, 6 links, 6 joints
Joints:
- joint legy: limit (none) -> lower=0

Commit message: added origins

File: hopper.urdf (robot description, URDF)
Before this commit: robot 2D_Hopper, 6 links, 6 joints
Joints:
- joint ground_is_world: origin (none) -> xyz=0 0 0
- joint legtheta: origin (none) -> xyz=0 0 0
- joint legx: origin (none) -> xyz=0 0 0
- joint legy: origin (none) -> xyz=0 0 0
